File: Eagle/SnapSat/mcuboard.brd (EAGLE design)
At the start: 80 x 80 mm, 6 parts

Commit message: extra breakouts
Parts:
- added THERMO1, THERMO2: (no value), pinhead:1X02
Connections:
- new net N$28: THERMO1.2, U$1.A0
- new net N$32: THERMO2.2, U$1.A1
- net N$9: now also THERMO1.1, THERMO2.1
Routing:
- net N$9: track 32.7 -> 78.7 mm, vias 0 -> 1
- net N$6: track 94.6 -> 131.4 mm
- net N$14: track 97.6 -> 123.4 mm, vias 1 -> 0
- net N$13: track 95.7 -> 120.5 mm
- net N$32: track 0.00 -> 23.5 mm
- net N$30: track 81.8 -> 102.3 mm
- net N$28: track 0.00 -> 20.1 mm
- net N$16: track 73.6 -> 93.3 mm, vias 1 -> 0
- net N$18: track 75.4 -> 57.2 mm
- net N$27: track 92.1 -> 76.2 mm
- net N$25: track 88.6 -> 73.2 mm
- net N$20: track 53.9 -> 68.4 mm, vias 0 -> 1
- net N$15: track 109.2 -> 122.2 mm
- net N$26: track 90.1 -> 78.2 mm
- net N$7: track 119.3 -> 108.9 mm
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