File: Eagle/SnapSat/mcuboard.sch (EAGLE design)
At the start: 6 parts

Commit message: extra breakouts
Parts:
- added THERMO1, THERMO2: (no value), pinhead:PINHD-1X2
Connections:
- new net N$28: THERMO1.2, U$1.A0_B
- new net N$32: THERMO2.2, U$1.A1
- net N$9: now also THERMO1.1, THERMO2.1
Changed lines of the file:
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@@
 <part name="R2" library="resistor" deviceset="R-EU_" device="0207_12"/>
 <part name="H" library="pinhead" deviceset="PINHD-2X8" device=""/>
+<part name="THERMO1" library="pinhead" deviceset="PINHD-1X2" device=""/>
+<part name="THERMO2" library="pinhead" deviceset="PINHD-1X2" device=""/>
 </parts>
 <sheets>
@@
 <instance part="R2" gate="G$1" x="5.08" y="73.66"/>
 <instance part="H" gate="A" x="149.86" y="33.02"/>
+<instance part="THERMO1" gate="G$1" x="-12.7" y="35.56"/>
+<instance part="THERMO2" gate="G$1" x="-12.7" y="22.86"/>
 </instances>
 <busses>
@@
 <segment>
 <pinref part="U$1" gate="G$1" pin="GND_A1"/>
-<wire x1="7.62" y1="45.72" x2="-17.78" y2="45.72" width="0.1524" layer="91"/>
+<wire x1="7.62" y1="45.72" x2="-5.08" y2="45.72" width="0.1524" layer="91"/>
+<wire x1="-5.08" y1="45.72" x2="-17.78" y2="45.72" width="0.1524" layer="91"/>
 <wire x1="-17.78" y1="45.72" x2="-17.78" y2="109.22" width="0.1524" layer="91"/>
 <wire x1="-17.78" y1="109.22" x2="111.76" y2="109.22" width="0.1524" layer="91"/>
@@
 <wire x1="111.76" y1="99.06" x2="121.92" y2="99.06" width="0.1524" layer="91"/>
 <junction x="7.62" y="45.72"/>
+<junction x="-5.08" y="45.72"/>
+<pinref part="THERMO1" gate="G$1" pin="1"/>
+<wire x1="-5.08" y1="38.1" x2="-5.08" y2="45.72" width="0.1524" layer="91"/>
+<wire x1="-15.24" y1="38.1" x2="-5.08" y2="38.1" width="0.1524" layer="91"/>
+<pinref part="THERMO2" gate="G$1" pin="1"/>
+<wire x1="-15.24" y1="25.4" x2="-20.32" y2="25.4" width="0.1524" layer="91"/>
+<wire x1="-20.32" y1="25.4" x2="-20.32" y2="45.72" width="0.1524" layer="91"/>
+<wire x1="-20.32" y1="45.72" x2="-17.78" y2="45.72" width="0.1524" layer="91"/>
+<junction x="-17.78" y="45.72"/>
+<junction x="-15.24" y="25.4"/>
+<junction x="-15.24" y="38.1"/>
 </segment>
 </net>
@@
 </segment>
 </net>
+<net name="N$28" class="0">
+<segment>
+<wire x1="-2.54" y1="35.56" x2="-2.54" y2="38.1" width="0.1524" layer="91"/>
+<wire x1="-2.54" y1="38.1" x2="7.62" y2="38.1" width="0.1524" layer="91"/>
+<pinref part="THERMO1" gate="G$1" pin="2"/>
+<wire x1="7.62" y1="38.1" x2="10.16" y2="38.1" width="0.1524" layer="91"/>
+<wire x1="-15.24" y1="35.56" x2="-2.54" y2="35.56" width="0.1524" layer="91"/>
+<junction x="-15.24" y="35.56"/>
+<pinref part="U$1" gate="G$1" pin="A0_B"/>
+<junction x="7.62" y="38.1"/>
+</segment>
+</net>
+<net name="N$32" class="0">
+<segment>
+<pinref part="THERMO2" gate="G$1" pin="2"/>
+<wire x1="-15.24" y1="22.86" x2="0" y2="22.86" width="0.1524" layer="91"/>
+<wire x1="0" y1="22.86" x2="0" y2="35.56" width="0.1524" layer="91"/>
+<pinref part="U$1" gate="G$1" pin="A1"/>
+<wire x1="0" y1="35.56" x2="7.62" y2="35.56" width="0.1524" layer="91"/>
+<junction x="-15.24" y="22.86"/>
+<junction x="7.62" y="35.56"/>
+</segment>
+</net>
